File: LiPo_Charger_1/LiPo_Charger_1.kicad_sch (KiCad schematic)
At the start: 21 parts

Commit message: 09.15 Update
Parts:
- removed J?: USB_MICRO-BREDUCED_PASTE, USB-B-MICRO-SMD_RED_PASTE, symbol SparkFun-Connectors:USB_MICRO-BREDUCED_PASTE
- added J1, J3: USB_B_Micro, Connector_USB:USB_Micro-B_Amphenol_10103594-0001LF_Horizontal, symbol Connector:USB_B_Micro
- added J2: Conn_01x02_Female, Connector_PinSocket_2.54mm:PinSocket_1x02_P2.54mm_Horizontal, symbol Connector:Conn_01x02_Female
- C1, C2, C3: renamed from C?; footprint (none) -> Capacitor_SMD:C_0201_0603Metric
- C4: renamed from C?; footprint (none) -> Capacitor_SMD:C_1812_4532Metric
- D1: renamed from D?; footprint DIOM6859X262N -> 403_charger:DIOM6859X262N
- D2, D3: renamed from D?; footprint (none) -> LED_SMD:LED_0201_0603Metric
- IC1: renamed from IC?; footprint SOT23-6 -> Package_TO_SOT_SMD:SOT-23-6
- L1: renamed from L?; footprint (none) -> Inductor_SMD:L_0805_2012Metric
- Q1: renamed from Q?; footprint lc_lib:SOT-23-6 -> Package_TO_SOT_SMD:SOT-23-6
- R1, R2, R3, R4, R5, R6, R7: renamed from R?; footprint (none) -> Resistor_SMD:R_0201_0603Metric
- SW1: renamed from SW?; footprint (none) -> Button_Switch_SMD:SW_DIP_SPSTx01_Slide_9.78x4.72mm_W8.61mm_P2.54mm
- gave numbers to parts that had none: 2
Connections:
- net 5V: now also J3.1 (VBUS)
- net BAT+: now also J2.1 (Pin_1)
- net BAT-: now also J2.2 (Pin_2)
- net GND: now also J1.5 (GND), J1.6 (Shield), J3.5 (GND), J3.6 (Shield)
- net OD: now reaches IC1.1 (OD), Q1.4 (G)
- net VBUS: now reaches C2.1, U1.4 (VCC), U1.8 (CE)
- net VBUS: now also J1.1 (VBUS)
- no-connect marks 3 -> 8
Other:
- note added: "Boost Circuit"
- note added: "Charging Circuit"
- note added: "Charging Port"
- note added: "OUT Port"
- note added: "Protection Circuit"
- moved on the sheet: C1, C2, C3, C4, D1, D2, D3, IC1, L1, Q1, R1, R2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

Commit message: 09/30/22
Parts:
- C1, C2: footprint Capacitor_SMD:C_0201_0603Metric -> lc_lib:0603_R
- C3: value 10u -> 22uF; footprint Capacitor_SMD:C_0201_0603Metric -> Capacitor_SMD:C_1206_3216Metric
- C4: footprint Capacitor_SMD:C_1812_4532Metric -> Capacitor_SMD:C_1206_3216Metric
- D1: value SS34_V7G -> SS34_mdd; footprint 403_charger:DIOM6859X262N -> 403_charger:SS34_mdd; symbol SS34_V7G:SS34_V7G -> 403-charger:SS34
- D2, D3: footprint LED_SMD:LED_0201_0603Metric -> lc_lib:0603_LED_S1
- J2: footprint Connector_PinSocket_2.54mm:PinSocket_1x02_P2.54mm_Horizontal -> Connector_PinHeader_1.00mm:PinHeader_1x02_P1.00mm_Vertical
- L1: footprint Inductor_SMD:L_0805_2012Metric -> 403_charger:75_75_4
- R1, R2, R3, R4, R5, R6, R7: footprint Resistor_SMD:R_0201_0603Metric -> lc_lib:0603_R
- SW1: footprint Button_Switch_SMD:SW_DIP_SPSTx01_Slide_9.78x4.72mm_W8.61mm_P2.54mm -> SW_500SSP3S1M6QEA; symbol Switch:SW_DIP_x01 -> 403-charger:500SSP3S1M6QEA; MANUFACTURER (none) -> E-Switch; MAXIMUM_PACKAGE_HEIGHT (none) -> 6.6 mm; PARTREV (none) -> D; SNAPEDA_PN (none) -> 500SSP1S1M6QEA; STANDARD (none) -> Manufacturer Recommendations
Connections:
- net BAT+: now also SW1.2; no longer SW1.1
- net at C3.1, L1.2, U2.4 (EN)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: now also SW1.3; no longer SW1.2
- no-connect marks 8 -> 9
Other:
- note added: "Battery Connection"
- title: (none) -> EE403W-Power Module
- moved on the sheet: J1, J3
